File: kicad/Solar_Array_Rev0/Solar_Array.sch (KiCad schematic (older format))
At the start: 27 parts, among them IC1 SPV1040, P1 PV_CELL, P2 CONN_01X07, Q1 Q_NPN_BCE, U1 LTC2990

Commit message: Organized for new Rev.
Parts:
- added D?: D_Schottky, symbol D_Schottky
- R5: value 12k -> 1k
- R6: value 1k2 -> 309
Connections:
- net at IC1.3 (LX), L1.1: now also D?.2 (A)
- net at C2.1, IC1.4 (VOUT), R2.1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: now also D?.1 (K)
Changed lines of the file:
@@
 P 5150 2600
 F 0 "R5" V 5230 2600 50  0000 C CNN
-F 1 "12k" V 5150 2600 50  0000 C CNN
+F 1 "1k" V 5150 2600 50  0000 C CNN
 F 2 "Resistors_SMD:R_0603" V 5080 2600 30  0001 C CNN
 F 3 "" H 5150 2600 30  0000 C CNN
@@
 P 5150 2900
 F 0 "R6" V 5230 2900 50  0000 C CNN
-F 1 "1k2" V 5150 2900 50  0000 C CNN
+F 1 "309" V 5150 2900 50  0000 C CNN
 F 2 "Resistors_SMD:R_0603" V 5080 2900 30  0001 C CNN
 F 3 "" H 5150 2900 30  0000 C CNN
@@
 F 0 "W1" H 2550 3410 50  0000 C CNN
 F 1 "TEST" H 2550 3280 50  0000 C CNN
-F 2 "Resistors_SMD:R_0805" H 2550 3350 50  0000 C CNN
+F 2 "Resistors_SMD:R_0805" H 2550 3550 50  0000 C CNN
 F 3 "" H 2550 3350 50  0000 C CNN
 	1    2550 3350
@@
 	1    0    0    -1
 $EndComp
+$Comp
+L D_Schottky D?
+U 1 1 56E8F7BD
+P 3400 2400
+F 0 "D?" H 3400 2500 50  0000 C CNN
+F 1 "D_Schottky" H 3400 2300 50  0000 C CNN
+F 2 "" H 3400 2400 50  0000 C CNN
+F 3 "" H 3400 2400 50  0000 C CNN
+	1    3400 2400
+	-1   0    0    1
+$EndComp
+Wire Wire Line
+	3250 2400 3150 2400
+Wire Wire Line
+	3150 2400 3150 2750
+Connection ~ 3150 2750
+Wire Wire Line
+	3550 2400 3900 2400
+Connection ~ 3900 2400
 $EndSCHEMATC
