File: MPPT/eagle/MPPT.sch (EAGLE design)
At the start: 1 part, among them U1 STM32F042K6

Commit message: Added Components for MPPT, started MPPT .brd .sch add TCAN330
Parts:
- added C1, C10, C12, C2, C4, C5, C6, C7, C8: NP, rcl_custom:C-EUC0603
- added C11, C16: 20p?, rcl_custom:C-EU0402-B-NOSILK
- added C15: 47u, rcl_custom:C-EUC0603
- added C17, C19, C22, C23, C3, C9: 100n, rcl_custom:C-EU0402-B-NOSILK
- added C20, C21: 4.7u, rcl:C-EUC0603
- added CF1: ORESAT-SOLARPANEL-12PIN, oresat-eagle:ORESAT-SOLARPANEL-12PIN
- added D2: ALTA-5-CELL-ARRAY, alta-cell:ALTA-5-CELL-ARRAY
- added D4: SOD123-B SCHOTTKY, apdm:DIODE_SCHOTTKY-SOD123-B
- added J1: 1.27MM-SWD-CONNECTOR, con-swd:1.27MM-SWD-CONNECTOR
- added L1: 10u, rcl:L-USL2012C
- added L2, L3: (no value), rcl:L-USL1812
- added Q1: ON-NFET, on-n-channel-fet:ON-N-CHANNEL-FET
- added Q2: P-CHANNELFET, vishay-p-channel-fet:P-CHANNELFET
- added R1: 10k, rcl_custom:R-US_0402-B-NOSILK
- added R13, R2: 100k, rcl_custom:R-US_0402-B-NOSILK
- added R14: 33.3k, rcl_custom:R-US_0402-B-NOSILK
- added R3: (no value), rcl:R-US_R0603
- added TP1, TP10, TP11, TP12, TP13, TP2, TP3, TP4, TP6, TP7, TP8, TP9: TEST-POINT, Tova:TEST-POINT
- added U$1: N-PMOSFET, N-PMosfet:N-PMOSFET
- added U$2: TSC888, TSC888:TSC888
- added U3: LM3671MF-3.3, LM3761:LM3761
- added U6: STM32F042K6, STM32F042K:STM32F042K6
- added X1: 8MHZ-2.5x2mm, low-gain-radio:CRYSTAL-WITH-GND
- U1: value STM32F042K6 -> TCAN330; device STM32F042K:STM32F042K6 -> TCAN330:TCAN330
Connections:
- new net 3.3V: C17.2, C19.1, C21.1, C22.2, C3.2, C9.2, J1.VTREF, L1.1, TP6.1, U$2.V+, U1.VCC, U3.FB, U6.VDD, U6.VDDA, U6.VDDIO2
- new net CANH: CF1.3, CF1.4, U1.CANH
- new net CANL: CF1.1, CF1.2, U1.CANL
- new net CAN_ENABLE: U1.SHDN, U6.PA10
- new net CAN_LSTN: U1.S, U6.PA9
- new net CAN_RX: U1.RXD, U6.PA11
- new net CAN_TX: U1.TXD, U6.PA12
- new net CRYSTALIN: C16.1, U6.PF0-OSC_IN, X1.1
- new net CRYSTALOUT: C11.1, U6.PF1-OSC_OUT, X1.2
- new net GND: C10.2, C11.2, C15.2, C16.2, C17.1, C19.2, C2.2, C20.2, C21.2, C22.1, C23.2, C3.1, C4.2, C5.2, C7.2, C9.1, CF1.10, CF1.9, D2.NEG, J1.GND, J1.GND@2, J1.GNDDET, L2.2, Q1.S, R14.1, U$1G$2.S, U$2.GND, U1.GND, U3.GND, U6.VSS, X1.SHIELD
- new net N$1: C1.1, C12.1, C6.1, C8.1, L2.1, U$1G$1.D
- new net N$10: TP13.1, U6.PB4
- new net N$11: C10.1, C15.1, C2.1, L3.1, R3.1, U$2.-IN
- new net N$12: U$1G$1.G, U6.PA1
- new net N$14: D4.ANODE, R3.2, U$2.+IN
- new net N$2: C1.2, C12.2, C6.2, C8.2, L3.2, U$1G$2.D
- new net N$3: CF1.6, TP1.1
- new net N$4: CF1.5, TP2.1
- new net N$5: TP8.1, U6.PA4
- new net N$6: TP9.1, U6.PA5
- new net N$7: TP10.1, U$2.OUT, U6.PA6
- new net N$8: TP11.1, U$1G$2.G, U6.PA7
- new net N$9: TP12.1, U6.PB3
- new net N6: Q1.D, Q2.G, R2.1
- new net ORESAT-SHDN: CF1.11, CF1.12, Q1.G, R1.1
- new net RESET: J1.!RESET, TP7.1, U6.NRST
- new net SOLAR-IN: D2.POS, Q2.S, R1.2, R2.2, TP3.1
- new net SOLAR-IN-SWITCHED: C20.1, C23.1, C4.1, C5.1, C7.1, Q2.D, R13.2, TP4.1, U$1G$1.S, U3.VIN
- new net STEPD: L1.2, U3.SW
- new net SWCLK: J1.SWDCLK/TCK, U6.PA14-SWCLK
- new net SWDIO: J1.SWDIO/TMS, U6.PA13-SWDIO
- new net VDIV: R13.1, R14.2, U3.EN
- new net VPV: CF1.7, CF1.8, D4.CATHODE
Other:
- note added: "1"
- note added: "Alta Devices 5 cell array - Voc = 5.45 V - Vmp = 4.80 V - Isc = 233 mA - Imp = 223 mA"
- note added: "N/C"
- note added: "NRST pull-up built in"
- note added: "OreSat Solar Module"
- note added: "Solar Module Shutdown"
- note added: "Turn on when EN > 1; with 1/3 divier, that's approximately 3.0V."
