File: zeta/eagle/MPPT.brd (EAGLE design)
At the start: 82 x 100 mm, 52 parts, among them J1 1.27MM-SWD-CONNECTOR, Q1 ON-NFET, Q2 P-CHANNELFET, U1 TCAN330, U3 LM3671MF-3.3, U6 STM32F042K6, X1 8MHZ-2.5x2mm

Commit message: Added Breakout Cable Schematic
Parts:
- C4: value NP -> 47u
Changed lines of the file:
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@@
 <attribute name="VALUE" x="19.225" y="77.705" size="0.635" layer="27" ratio="20" rot="R270"/>
 </element>
-<element name="C4" library="rcl_custom" package="C0603" value="NP" x="29.1" y="62.8" smashed="yes" rot="R180">
+<element name="C4" library="rcl_custom" package="C0603" value="47u" x="29.1" y="62.8" smashed="yes" rot="R180">
 <attribute name="NAME" x="26.2" y="63.05" size="0.635" layer="25" font="vector" ratio="20" rot="R180"/>
 <attribute name="VALUE" x="29.9" y="65.1" size="0.635" layer="27" ratio="20" rot="R180"/>
