File: 1u_panel/eagle/1u_panel_v1.1.sch (EAGLE design)
At the start: 59 parts, among them Q3 MMBT3904, U2 TCAN330, U3 LM3671MF-3.3, U4 ZSPM4521, U5 LTC2990, U6 STM32F042K6, X1 16MHZ-2.5x2mm

Commit message: First version of the 1.1 solar panel. Keeping 1.0 for future reference.
Parts:
- added TP16, TP17, TP18, TP19, TP20, TP21, TP22, TP23: TEST-POINT, Tova:TEST-POINT
- added U1, U7, U8, U9: LTC4411, ltc4411:LTC4411
- D3: value STPS1L40AY -> DNP/STPS1L40AY
Connections:
- net N$13 renamed ZSPM_EN
- new net N$12: U1.OUT, U7.IN
- new net N$15: U8.OUT, U9.IN
- new net N$16: TP16.1, U1.STAT
- new net N$17: TP23.1, U9.CTL
- new net N$18: TP17.1, U7.STAT
- new net N$19: TP18.1, U9.STAT
- new net N$20: TP19.1, U8.STAT
- new net N$21: TP22.1, U7.CTL
- new net N$22: TP21.1, U1.CTL
- new net N$23: TP20.1, U8.CTL
- net GND: now also U1.GND, U7.GND, U8.GND, U9.GND
- net VPV: now also U7.OUT, U9.OUT
- net VSOLAR: now also U1.IN, U8.IN
Other:
- note removed: "~4.9V"
- moved on the sheet: C1, C11, C14, C16, C17, C18, C19, C2, C20, C21, C22, C23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
