File: 1u_panel/kicad/1u_panel-microcontroller.kicad_sch (KiCad schematic)
At the start: 43 parts, among them J2 2-1734592-0, U1 TCAN330GDCNT, U11 TMP101NA/3KSLOTTED, U2 TMP101NA/3KSLOTTED, U7 STM32F091CCT7, X1 ECS-160-10-36Q-ES-TR

Commit message: Beginning of the v6.0 solar boards. Lots of ways to go.
Parts:
- J2: footprint 1u_panel:TE_2-1734592-0 -> oresat-connectors:J-TE-2-1734592-0; symbol 1u_panel-eagle-import:ORESAT-DEBUG-CONNECTOR-ALL -> oresat-connectors:J-TE-2-1734592-0
Other:
- note removed: "5"
- note removed: "OreSat Solar Board: Microcontroller"
- title: (none) -> OreSat Solar Module (for Frame 2.0)
- moved on the sheet: C1, C11, C16, C25, C26, C27, C28, C29, C3, C30, C31, C5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
