File: 1u_panel/kicad/1u_panel-power.kicad_sch (KiCad schematic)
At the start: 69 parts, among them J1 MMS-104-01-[F/L]-SH, Q1 DMP3050LVT-7, Q2 DMP2240UDM-7, U10 TPS63060DSCR, U12 LTC4412, U3 LT1618EMSTRPBF, U4 INA226AIDGSR

Commit message: Fixed R12 value to make VOUT to 8.4V max. Was at 8.6V max. Also cleaned up some EAGLE import issues, mostly text size and labels.
Parts:
- R12: value 14.2k -> 14.7k
Other:
- note added: "All caps are ceramic 10% X5R >= 16V Vwv and AEQ unless marked"
- note added: "All resistors 0603 +/- 1% and AEQ unless marked"
- note added: "Asserts ~{SD}."
- note added: "Fiducials"
- note added: "Make 8.35V max"
- note added: "Requires 2mm male shorting plug."
- note removed: "All caps are ceramic 10% X5R >= 16V Vwv unless marked"
- note removed: "All resistors 0603 +/- 1% unless marked"
- note removed: "ONLY POPULATED IN +Z+X SOLAR BOARD. DNP ALL OTHER BOARDS. Requires 2mm male shorting plug."

Commit message: Beginning of the v6.0 solar boards. Lots of ways to go.
Other:
- note removed: "5.1"
- note removed: "OreSat Solar Board: MPPT + PWR"
- title: (none) -> OreSat Solar Module (for Frame 2.0)
- moved on the sheet: C12, C13, C14, C15, C18, C19, C2, C20, C21, C22, C23, C4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
