File: 1u_panel_silicon_cells/kicad/1u_panel-silicon.kicad_sch (KiCad schematic)
At the start: 0 parts

Commit message: fixed board outline, title blocks
Other:
- title: OreSat Solar Module (for Frame 2.0) -> OreSat Silicon Solar Module (for Frame 2.0)
Changed lines of the file:
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@@
 	(paper "USLedger")
 	(title_block
-		(title "OreSat Solar Module (for Frame 2.0)")
-		(date "2023-12-20")
-		(rev "6.0")
+		(title "OreSat Silicon Solar Module (for Frame 2.0)")
+		(date "2024-08-18")
+		(rev "1.0")
 	)
 	(sheet

Commit message: Polish on Jack's final design. Swapped out rectangles for zones on multiple layers, cleaned up a lot of small layout bits, fixed some mechanical crashes with screw heads, fixed up the silk screen, and added 3D models.
Other:
- title: OreSat Silicon Solar Module (for Frame 2.0) -> OreSat Solar Module - Silicon Cells
Changed lines of the file:
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@@
 	(paper "USLedger")
 	(title_block
-		(title "OreSat Silicon Solar Module (for Frame 2.0)")
-		(date "2024-08-18")
+		(title "OreSat Solar Module - Silicon Cells")
+		(date "2024-09-22")
 		(rev "1.0")
 	)
