File: 1u_panel_silicon_cells/solar-module-1u-si.kicad_pcb (KiCad board)
At the start: 2 copper layers, 83 x 100 mm, 143 parts, among them J1 MMS-104-01-[F/L]-SH, J2 2-1734592-0, Q1 NTR4101P, Q2 DMP2240UDM-7, U1 TCAN330, U10 TPS63060DSCR, U11 TMP101NA/3KSLOTTED, U12 LTC4412, U13 LTC4411, U14 LTC4411, U15 LTC4411, U16 LTC4411, U2 TMP101NA/3KSLOTTED, U3 LT1618EMSTRPBF, U4 INA226, U5 LTC4411, U6 LTC4411, U7 STM32F091CCT7, U8 LTC4411, U9 LTC4411, X1 ECS-160-10-36Q-ES-TR

Commit message: Yeah, renamed everything because consistancy.
Connections:
- net /1u_panel-microcontroller/BOOT0 renamed /Microcontroller/BOOT0
- net /1u_panel-microcontroller/CAN_RX renamed /Microcontroller/CAN_RX
- net /1u_panel-microcontroller/CAN_SHDN renamed /Microcontroller/CAN_SHDN
- net /1u_panel-microcontroller/CAN_SILENT renamed /Microcontroller/CAN_SILENT
- net /1u_panel-microcontroller/CAN_TX renamed /Microcontroller/CAN_TX
- net /1u_panel-microcontroller/NRESET renamed /Microcontroller/NRESET
- net /1u_panel-microcontroller/OSC_IN renamed /Microcontroller/OSC_IN
- net /1u_panel-microcontroller/OSC_OUT renamed /Microcontroller/OSC_OUT
- net /1u_panel-microcontroller/PA0 renamed /Microcontroller/PA0
- net /1u_panel-microcontroller/PA2/USART2_TX renamed /Microcontroller/PA2/USART2_TX
- net /1u_panel-microcontroller/PA3/USART2_RX renamed /Microcontroller/PA3/USART2_RX
- net /1u_panel-microcontroller/SWCLK renamed /Microcontroller/SWCLK
- net /1u_panel-microcontroller/SWDIO renamed /Microcontroller/SWDIO
- net /1u_panel-power/TPS-VOUT-3.3V renamed /MPPT and Power/TPS-VOUT-3.3V
- net /1u_panel-power/VMPPT renamed /MPPT and Power/VMPPT
- net /1u_panel-power/~{SHDN-3.3V} renamed /MPPT and Power/~{SHDN-3.3V}
- net /1u_panel-power/~{SHDN-OUPUT} renamed /MPPT and Power/~{SHDN-OUPUT}
- net /1u_panel-power/~{SHUTDOWN} renamed /MPPT and Power/~{SHUTDOWN}
