File: solar-module-1u-si-MCXN/solar-module-1u-si.kicad_sch (KiCad schematic)
At the start: 6 parts

Commit message: Final polishing before fab. Fixed I2C pullups, removed some silly test points, lots of good zone planning on layer 3, cleaned up solar ideal diodes, moved LED to a blink light instead of power light.
Other:
- title: OreSat Solar Module - Silicon Cells -> OreSat Solar Module - Silicon Cells + MCXN
Changed lines of the file:
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@@
 	(paper "USLedger")
 	(title_block
-		(title "OreSat Solar Module - Silicon Cells")
-		(date "2025-09-16")
+		(title "OreSat Solar Module - Silicon Cells + MCXN")
+		(date "2025-09-23")
 		(rev "1.1")
 	)
