File: solar-module-1u-si-MCXN/solar-module-1u-si-sch-cells.kicad_sch (KiCad schematic)
At the start: 41 parts, among them U13 LTC4411, U14 LTC4411, U15 LTC4411, U16 LTC4411, U5 LTC4411, U6 LTC4411, U8 LTC4411, U9 LTC4411

Commit message: Final polishing before fab. Fixed I2C pullups, removed some silly test points, lots of good zone planning on layer 3, cleaned up solar ideal diodes, moved LED to a blink light instead of power light.
Other:
- title: OreSat Solar Module - Silicon Cells -> OreSat Solar Module - Silicon Cells + MCXN
Changed lines of the file:
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@@
 	(paper "USLedger")
 	(title_block
-		(title "OreSat Solar Module - Silicon Cells")
-		(date "2025-09-16")
+		(title "OreSat Solar Module - Silicon Cells + MCXN")
+		(date "2025-09-23")
 		(rev "1.1")
 	)

Commit message: Fix up BOM
Parts:
- C10, C39, C40, C41, C42, C43, C44, C45: DIS Digi-Key -> DigiKey; DPN 1276-1784-1-ND -> 587-4332-1-ND; MFR Samsung Electro-Mechanics -> Taiyo Yuden; MPN CL10A475KO8NNNC -> EMK107BBJ475KAHT
- C17, C24, C32, C33, C34, C35, C36, C38: DIS Digi-Key -> DigiKey
- D10, D11, D12, D13, D2, D7, D8, D9, U13, U14, U15, U16, U5, U6, U8, U9: DIS Digi-Key -> DIgiKey
