File: 1u-solar-breakout/1u-solar-breakout.kicad_pcb (KiCad board)
At the start: 2 copper layers, 1 part

Commit message: layout made (needs a design review)
Parts:
- added J3: 302-S201, Connector_IDC:IDC-Header_2x10_P2.54mm_Vertical, F.Cu at (501.2, 195.6)
- added TP2: TEST-POINT-LARGE-SQUARE, oresat-misc:TestPoint-0.75mm-th, F.Cu at (482.5, 202.5)
- moved CF1 41.5 mm to (489.0, 203.0), turned to 90 degrees
Routing:
- net Net-(J3-Pin_17): track 0.00 -> 26.8 mm
- net Net-(J3-Pin_13): track 0.00 -> 25.5 mm
- net Net-(J3-Pin_10): track 0.00 -> 23.9 mm
- net Net-(J3-Pin_1): track 0.00 -> 23.3 mm
- net Net-(J3-Pin_5): track 0.00 -> 22.8 mm
- net (no net): track 0.00 -> 9.80 mm
- net Net-(CF1-AUX-Pad7): track 0.00 -> 3.81 mm

Commit message: final revisions made (ready for design review!)
Parts:
- moved TP2 337.9 mm to (161.5, 97.0)
- moved CF1 334.3 mm to (172.8, 94.6)
- moved J3 331.4 mm to (187.2, 89.6)
Routing:
- net Net-(CF1-AUX-Pad7): track 3.81 -> 15.3 mm
- net (no net): track 9.80 -> 0.00 mm
- net Net-(J3-Pin_17): track 26.8 -> 30.2 mm
- net Net-(J3-Pin_5): track 22.8 -> 25.7 mm
- net Net-(J3-Pin_13): track 25.5 -> 28.3 mm
- net Net-(J3-Pin_10): track 23.9 -> 26.7 mm
- net Net-(J3-Pin_1): track 23.3 -> 25.6 mm

Commit message: initial review made (still needs official review from andrew)
Parts:
- J3: moved to B.Cu
- TP2: footprint oresat-misc:TestPoint-0.75mm-th -> oresat-misc:TestPoint_Pad_D1.0mm
- moved TP2 17.2 mm to (177.0, 104.5), turned to 180 degrees
- moved CF1 5.25 mm to (178.0, 94.6)
- moved J3 3.78 mm to (190.5, 87.7), turned to 180 degrees
Connections:
- net Net-(J3-Pin_13) renamed GND
Routing:
- net GND: track 28.3 -> 0.00 mm
- net Net-(J3-Pin_5): track 25.7 -> 20.4 mm
- net Net-(J3-Pin_10): track 26.7 -> 21.4 mm
- net Net-(CF1-AUX-Pad7): track 15.3 -> 20.1 mm
- net Net-(J3-Pin_1): track 25.6 -> 20.8 mm
- net Net-(J3-Pin_17): track 30.2 -> 26.4 mm
- added copper zone on B.Cu, net GND
- added copper zone on F.Cu, net GND
Other:
- board outline added: 24 x 37 mm
