File: 1u-solar-breakout/1u-solar-breakout.kicad_sch (KiCad schematic)
At the start: 3 parts, among them J3 302-S201

Commit message: final revisions made (ready for design review!)
Other:
- company: (none) -> oresat!
- title: (none) -> 1u Solar Breakout
Changed lines of the file:
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@@
 	(generator_version "10.0")
 	(paper "A4")
+	(title_block
+		(title "1u Solar Breakout")
+		(date "2026-09-15")
+		(rev "0")
+		(company "oresat!")
+	)
 	(junction
 		(at 173.99 109.22)

Commit message: initial review made (still needs official review from andrew)
Parts:
- TP2: footprint oresat-misc:TestPoint-0.75mm-th -> oresat-misc:TestPoint_Pad_D1.0mm
Connections:
- net GND: now also CF1.3 (GND), CF1.4 (GND), J3.13 (Pin_13), J3.14 (Pin_14), J3.15 (Pin_15), J3.16 (Pin_16); no longer CF1.P$1 (SHIELD), CF1.P$2 (SHIELD), CF1.P$3 (SHIELD), CF1.P$4 (SHIELD)
- new net: CF1.P$1 (SHIELD), CF1.P$2 (SHIELD), CF1.P$3 (SHIELD), CF1.P$4 (SHIELD)
- no-connect marks 0 -> 1
Changed lines of the file:
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@@
+	)
+	(junction
+		(at 194.31 66.04)
+		(diameter 0)
+		(color 0 0 0 0)
 	)
 	(junction
@@
 		(color 0 0 0 0)
 	)
-	(wire
-		(pts
-			(xy 205.74 66.04) (xy 181.61 66.04)
+	(no_connect
+		(at 208.28 81.28)
+	)
+	(wire
+		(pts
+			(xy 205.74 66.04) (xy 194.31 66.04)
 		)
 		(stroke
@@
 	(wire
 		(pts
-			(xy 208.28 81.28) (xy 208.28 83.82)
+			(xy 194.31 66.04) (xy 194.31 82.55)
 		)
 		(stroke
@@
 		(pts
 			(xy 186.69 73.66) (xy 205.74 73.66)
+		)
+		(stroke
+			(width 0)
+			(type default)
+		)
+	)
+	(wire
+		(pts
+			(xy 194.31 66.04) (xy 181.61 66.04)
 		)
 		(stroke
@@
 			)
 		)
-		(property "Footprint" "oresat-misc:TestPoint-0.75mm-th"
+		(property "Footprint" "oresat-misc:TestPoint_Pad_D1.0mm"
 			(at 191.77 60.96 0)
 			(hide yes)
@@
 	(symbol
 		(lib_id "power:GND")
-		(at 208.28 83.82 0)
+		(at 194.31 82.55 0)
 		(unit 1)
 		(body_style 1)
@@
 		(fields_autoplaced yes)
 		(property "Reference" "#PWR01"
-			(at 208.28 90.17 0)
+			(at 194.31 88.9 0)
 			(hide yes)
 			(show_name no)
@@
 		)
 		(property "Value" "GND"
-			(at 208.28 88.9 0)
+			(at 194.31 87.63 0)
 			(show_name no)
 			(do_not_autoplace no)
@@
 		)
 		(property "Footprint" ""
-			(at 208.28 83.82 0)
+			(at 194.31 82.55 0)
 			(hide yes)
 			(show_name no)
@@
 		)
 		(property "Datasheet" ""
-			(at 208.28 83.82 0)
+			(at 194.31 82.55 0)
 			(hide yes)
 			(show_name no)
@@
 		)
 		(property "Description" "Power symbol creates a global label with name \"GND\" , ground"
-			(at 208.28 83.82 0)
-			(hide yes)
-			(show_name no)
+			(at 194.31 82.55 0)
+			(hide yes)
+			(show_name no)
